Commit message: hmw3

File: ros2_iiwa/iiwa_description/urdf/arm_camera.xacro (robot description, xacro)
@@ -5,12 +5,12 @@
     <sensor name="camera" type="camera">
         <camera>
-        <horizontal_fov>1.047</horizontal_fov>
+        <horizontal_fov>1.089</horizontal_fov>
         <image>
-            <width>320</width>
-            <height>240</height>
+            <width>620</width>
+            <height>480</height>
         </image>
         <clip>
-            <near>0.1</near>
-            <far>100</far>
+            <near>0.05</near>
+            <far>8.0</far>
         </clip>
         </camera>

File: ros2_iiwa/iiwa_description/urdf/iiwa.urdf.xacro (robot description, xacro)
@@ -244,9 +244,15 @@
         <inertia ixx="0.05"  ixy="0"  ixz="0" iyy="0.018" iyz="0" izz="0.044" />
       </inertial>
-  </link>
+    </link>
+    <link name="camera_link_optical"></link>
     <joint name="camera_joint" type="fixed">
       <parent link="${prefix}tool0"/>
       <child link="camera_link"/>
       <origin xyz="0 0 0" rpy="0 -1.57 3.14"/>
+    </joint>
+    <joint name="camera_optical_joint" type="fixed">
+      <parent link="camera_link"/>
+      <child link="camera_link_optical"/>
+      <origin xyz="0 0 0" rpy="${-pi/2} 0 ${-pi/2}"/>
     </joint>
     <xacro:include filename="$(find iiwa_description)/urdf/arm_camera.xacro"/>
